File: PCB Eagle/buisiness_card.brd (EAGLE design)
At the start: 85 x 54 mm, 24 parts, among them Y1 16MHz

Commit message: Added BOM and updated components references.
Parts:
- renumbered U$10 to B8, U$11 to B7, U$12 to B10, U$13 to B9, U$2 to U1, U$3 to U2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
